File: hardware/pcb/dev-board/dev-board.kicad_pcb (KiCad board)
At the start: 2 copper layers, 64.9 x 66.2 mm, 24 parts, among them J1 Conn_01x04, J2 Conn_01x04, J3 Conn_01x04, J4 Conn_01x04, J5 CON-SOCJ-2155, J6 UART, J7 Conn_01x03, J8 Conn_01x11, U1 Pico, U2 L7805

Commit message: Finished dev board PCB
Parts:
- added FID1: Fiducial, Fiducial:Fiducial_1mm_Mask2mm, F.Cu at (131.4, 50.4)
- added FID2: Fiducial, Fiducial:Fiducial_1mm_Mask2mm, F.Cu at (192.5, 112.2)
- added FID3: Fiducial, Fiducial:Fiducial_1mm_Mask2mm, F.Cu at (175.4, 60.1)
- J1: value Conn_01x04 -> Motor 1
- J4: renamed from J2; value Conn_01x04 -> Motor 3
- J5: renamed from J3; value Conn_01x04 -> Motor 2
- J6: renamed from J4; value Conn_01x04 -> Motor 4
- J8: renamed from J7; value Conn_01x03 -> DEBUG
- moved C5 1.75 mm to (174.1, 105.6)
- moved C6 1.75 mm to (167.4, 105.6)
- moved U2 1.75 mm to (173.3, 109.0)
- moved J2 1.10 mm to (189.5, 53.0)
- moved J8 1.10 mm to (189.5, 94.2)
- moved J7 0.74 mm to (186.3, 109.0)
- renumbered C4 to C3, C3 to C4, C6 to C5, C5 to C6, J6 to J2, J8 to J3, J5 to J7, R3 to R2, R2 to R3
Routing:
- net +5V: track 235.5 -> 182.8 mm
- net /M2: track 51.5 -> 74.4 mm
- net GND: track 80.1 -> 97.9 mm, vias 38 -> 57
- net VDC: track 105.2 -> 110.1 mm
- net Net-(J2-Pin_3): track 33.0 -> 31.2 mm
- net /M4_STEP: track 27.1 -> 28.3 mm
- net /M2_STEP: track 29.5 -> 30.7 mm
- net Net-(J8-Pin_1): track 20.4 -> 19.3 mm
- net Net-(J8-Pin_2): track 23.2 -> 22.1 mm
- net /M1_STEP: track 37.2 -> 38.1 mm
- net /M3_STEP: track 27.1 -> 27.7 mm
- net /M1_DIR: track 39.9 -> 40.4 mm
Other:
- board text added: "+5V"
- board text added: "GND"
- board text added: "GP17"
- board text added: "GP18"
- board text added: "GP19"
- board text added: "GP20"
- board text added: "GP21"
- board text added: "GP22"
- board text added: "GP26"
- board text added: "GP27"
- board text added: "GP28"
- board text added: "Stepper Dev Board, V1.0"
