File: hardware/pcb/dev-board/dev-board.kicad_sch (KiCad schematic)
At the start: 24 parts, among them J1 Conn_01x04, J2 CON-SOCJ-2155, J2 Conn_01x04, J3 Conn_01x04, J4 Conn_01x04, J6 UART, J7 Conn_01x03, J8 Conn_01x11, U1 Pico, U2 L7805

Commit message: Finished dev board PCB
Parts:
- added FID1, FID2, FID3: Fiducial, Fiducial:Fiducial_1mm_Mask2mm, symbol Mechanical:Fiducial
- J1: value Conn_01x04 -> Motor 1
- J4: renamed from J2; value Conn_01x04 -> Motor 3
- J5: renamed from J3; value Conn_01x04 -> Motor 2
- J6: renamed from J4; value Conn_01x04 -> Motor 4
- renumbered C6 to C5, C5 to C6, J6 to J2, J8 to J3, J7 to J8, R3 to R2, R2 to R3
Connections:
- no-connect marks 4 -> 5
Other:
- moved on the sheet: C5, C6, J2, J3, U2
