File: hardware/pcb/tentacle-board/tentacle-board.kicad_pcb (KiCad board)
At the start: 2 copper layers, 48.4 x 54.9 mm, 80 parts, among them IC1 W25Q32JVZPIQ, J1 Motor, J2 AUX2, J3 UART0, J4 Motor, J5 AUX1, J6 DEBUG, J7 CTRL, J8 Conn_01x02, U1 DRV8825PWP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

Commit message: Updated the firmware project to build the custom board. Fixed some missing silkscreen items on the pcb.
Other:
- rule pad_to_mask_clearance: 0.051 -> 0
Changed lines of the file:
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@@
   )
   (setup
-    (pad_to_mask_clearance 0.051)
-    (solder_mask_min_width 0.09)
+    (pad_to_mask_clearance 0)
     (aux_axis_origin 100 100)
     (grid_origin 121.59 74)
@@
       (psa4output false)
       (plotreference true)
-      (plotvalue false)
+      (plotvalue true)
       (plotinvisibletext false)
       (sketchpadsonfab false)
-      (subtractmaskfromsilk true)
+      (subtractmaskfromsilk false)
       (outputformat 1)
       (mirror false)
       (drillshape 0)
       (scaleselection 1)
-      (outputdirectory "gerbers")
+      (outputdirectory "release-v1.1")
     )
   )
